File: filters.sch (KiCad schematic (older format))
At the start: 0 parts

Commit message: Updates to the filter page
Added a blackrock_components that just has some new parts
Parts:
- added C? (x2): 0.1uF, ~, symbol C
- added C? (x2): 0.047uF, ~, symbol C
- added C? (x3): 680pF, ~, symbol C
- added C? (x2): 1500pF, ~, symbol C
- added C? (x3): 390pF, ~, symbol C
- added C? (x2): 180pF, ~, symbol C
- added C? (x2): 100pF, ~, symbol C
- added J?: SMA, sma, symbol SMA
- added JP?: JUMPER, ~, symbol JUMPER
- added L? (x2): 5.5uH, symbol L
- added L?: 2.6uH, symbol L
- added L? (x2): 2uH, symbol L
- added L? (x3): 0.46uH, symbol L
- added L? (x2): 1uH, symbol L
- added L?: 0.27uH, symbol L
- added L?: 0.13uH, symbol L
- added R? (x2): 2.2k, ~, symbol R
- added R? (x2): 120, ~, symbol R
- added R? (x4): 75, ~, symbol R
- added T?: TRANSFO, ~, symbol TRANSFO
- added U?: FST3253, TSSOP16, symbol FST3253
Connections:
- net labels added: +5V, AGND, ft_sel_0, ft_sel_1
- wire segments 0 -> 69
Other:
- note added: "BAND 0"
- note added: "BAND 1"
- note added: "BAND 2"
- note added: "BAND 3"

Commit message: Finished filters page, started demod
Parts:
- added C?: 0.1uF, ~, symbol C
- added U?: FST3253, TSSOP16, symbol FST3253
Connections:
- net labels added: ft_ana
- wire segments 69 -> 120
Other:
- note added: "FIGURE OUT THIS CONNECTOR"
- moved on the sheet: C?, JP?, L?, R?, T?, U?
